Commit message: Added the other joints of our 3D Model to the movit config

File: config/hand.xacro (robot description, xacro)
@@ -12,4 +12,9 @@
       <link name="panda_rightfinger" />
       <joint name="panda_finger_joint1" />
+      <link name="panda_realsense_hole_1"/>
+      <link name="panda_realsense_hole_2"/>
+      <link name="panda_realsense_hole_3"/>
+      <link name="panda_realsense_hole_4"/>
+      <link name="panda_aruco_center"/>
       <passive_joint name="panda_finger_joint2" />
     </group>
